File: kicad/can.sch (KiCad schematic (older format))
At the start: 11 parts, among them U5 TCAN334

Commit message: License update and larger inductor (v0.2.3)
- Change license to CERN-OHL-W-2.0, which is more suitable for hardware
- Use larger nominal 53 uH inductor to support 20A also for 24V systems
- Increase input capacitor height to 25 mm (inductor needs more space anyway)
- Update schematic template and text fields
- Use photo instead of rendered image
Parts:
- JP1: symbol Device:Jumper_NC_Small -> LibreSolar:Jumper_NC_Small
Changed lines of the file:
@@
 Title "MPPT 2420 HC"
 Date "2021-01-06"
-Rev "0.2.2"
-Comp "Libre Solar Technologies GmbH"
-Comment1 "https://libre.solar"
+Rev "0.2.3"
+Comp "Copyright © 2020 Libre Solar Technologies GmbH"
+Comment1 "Licensed under CERN-OHL-W version 2"
 Comment2 "Author: Martin Jäger"
-Comment3 "License: Creative Commons Attribution-ShareAlike 4.0 International"
+Comment3 ""
 Comment4 ""
 $EndDescr
@@
 $EndComp
 $Comp
-L Device:Jumper_NC_Small JP1
+L LibreSolar:Jumper_NC_Small JP1
 U 1 1 5E3006CE
 P 4700 3500
+AR Path="/5E3006CE" Ref="JP1"  Part="1"
+AR Path="/5F16179B/5E3006CE" Ref="JP1"  Part="1"
 F 0 "JP1" V 4654 3574 50  0000 L CNN
 F 1 "Jumper_NC_Small" V 4745 3574 50  0000 L CNN
